File: CONFIG.kicad_sch (KiCad schematic)
At the start: 32 parts, among them SW1 SW_SPST, U12 OSC_100M, U2 ICE40HX8K-BG121, U4 TPS74633, U5 TPS74612, U6 W25Q32JVSS, U9 TPS74618

Commit message: Routing changes, pullups, etc
Parts:
- added J4: Conn_01x04, Connector_Molex:Molex_CLIK-Mate_502382-0970_1x09-1MP_P1.25mm_Vertical, symbol Connector_Generic:Conn_01x09
- added R25, R26, R27: 10k, Resistor_SMD:R_0402_1005Metric, symbol Device:R
- C14, C15, C16, C17, C18, C19, C23, C24, C25, C27, C28, C29, C31, C32, C33, D10, D6, D7, D8, D9, JP1, R13, R14, R20, SW1, U2, U4, U5, U6, U9: Source (none) -> ANY
- R15: value R -> 10k; Source (none) -> ANY
- U12: value OSC_100M -> ASEMB-100.000MHZ-LY-T; Source (none) -> ANY
Connections:
- net +1V2: now also R26.2, R27.2; no longer C16.1, C17.1, U2.C6 (VCCPLL1), U2.J6 (VCCPLL0)
- net GND: now also J4.1 (Pin_1)
- net VCC: now also J4.2 (Pin_2), R25.1
- net at U2.K10 (IOB_108_SS), U6.1 (~CS): now also J4.7 (Pin_7), R25.2
- net at U2.J9 (IOB_106_SDI), U6.2 (DO(IO1)): now also J4.5 (Pin_5)
- net at U2.K9 (IOB_105_SDO), U6.5 (DI(IO0)): now also J4.6 (Pin_6)
- net at U2.L10 (IOB_107_SCK), U6.6 (CLK): now also J4.8 (Pin_8)
- net DBG_AUX_A: now reaches U2.K3 (IOB_63)
- net DBG_AUX_A: now also J4.3 (Pin_3)
- net DBG_AUX_B: now reaches U2.K4 (IOB_73)
- net DBG_AUX_B: now also J4.4 (Pin_4)
- net CRESET renamed ~CRESET
- net ~CRESET: now also J4.9 (Pin_9)
- new net: C17.1, R27.1, U2.C6 (VCCPLL1)
- new net: C16.1, R26.1, U2.J6 (VCCPLL0)
Other:
- note added: "ANY"
- moved on the sheet: C14, C15, C18, C19, C23, C24, C25, C27, C28, D10, D6, D7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

Commit message: Routing cleanup, fix primary transformer
Parts:
- added C40: C, Capacitor_SMD:C_0402_1005Metric, symbol Device:C
- added R28: 10k, Resistor_SMD:R_0402_1005Metric, symbol Device:R
- J4: value Conn_01x04 -> 502382-0970
- SW1: value SW_SPST -> 434133025816
Connections:
- net GND: now also C40.2
- net VCC: now also C40.1, R28.1
- net at J4.8 (Pin_8), U2.L10 (IOB_107_SCK), U6.6 (CLK): now also R28.2
Other:
- note removed: "ANY"
- moved on the sheet: C14, C15, C16, C17, C18, C19, C23, C24, C25, C27, C28, C29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
